File: BodyComputer/BodyComputer/BodyComputer.sch (KiCad schematic (older format))
At the start: 0 parts

Commit message: Body Computer - 4layer
Added 4-layer board layout, changed schematic a bit, added jumper for NodeMCU powering, control MOSFET for Fans
Changed lines of the file:
@@
 Sheet 1 7
 Title "Body Computer"
-Date "2020-04-01"
+Date "2020-04-12"
 Rev "1.0"
 Comp "Wojciech Grzeliński"
@@
 $EndSheet
 $Sheet
-S 8500 1000 1000 2000
+S 8500 1000 1000 2150
 U 5E6DC799
 F0 "Peripherals" 50
@@
 F16 "LCD_SCL" I L 8500 2800 50
 F17 "RESET_BUTTON" I L 8500 2950 50
+F18 "FAN_CONTROL" I L 8500 3100 50
 $EndSheet
 $Sheet
@@
 Wire Wire Line
 	8500 1300 7500 1300
+Wire Wire Line
+	8500 1600 7500 1600
+Wire Wire Line
+	7500 1700 8500 1700
+Wire Wire Line
+	8500 1850 7500 1850
+Wire Wire Line
+	7500 1950 8500 1950
+Wire Wire Line
+	8500 2100 7500 2100
+Wire Wire Line
+	7500 2200 8500 2200
+Wire Wire Line
+	8500 2300 7500 2300
+Wire Wire Line
+	7500 2450 8500 2450
+Wire Wire Line
+	8500 2550 7500 2550
+Wire Wire Line
+	8500 3600 7500 3600
+Wire Wire Line
+	7500 3700 8500 3700
+Wire Wire Line
+	8500 2700 7500 2700
+Wire Wire Line
+	7500 2800 8500 2800
+Wire Wire Line
+	8500 1100 7500 1100
+Wire Wire Line
+	5000 2750 3500 2750
+Wire Wire Line
+	5000 2850 3500 2850
+Wire Wire Line
+	8500 5650 7500 5650
+Wire Wire Line
+	7500 5550 8500 5550
+Wire Wire Line
+	8500 5450 7500 5450
+Wire Wire Line
+	7500 5350 8500 5350
+Wire Wire Line
+	8500 5100 7500 5100
+Wire Wire Line
+	7500 5000 8500 5000
+Wire Wire Line
+	8500 4900 7500 4900
+Wire Wire Line
+	7500 4800 8500 4800
+Wire Wire Line
+	8500 4700 7500 4700
+Wire Wire Line
+	7500 4600 8500 4600
+Wire Wire Line
+	8500 3950 7500 3950
+Wire Wire Line
+	7500 3850 8500 3850
+Wire Wire Line
+	5000 3350 3500 3350
+Wire Wire Line
+	3500 3450 5000 3450
+Wire Wire Line
+	5000 3550 3500 3550
+Wire Wire Line
+	3500 3650 5000 3650
+Wire Wire Line
+	5000 3750 3500 3750
+Wire Wire Line
+	3500 3850 5000 3850
+Wire Wire Line
+	8500 2950 7500 2950
+$Sheet
+S 2500 4350 1000 1650
+U 5F25F1A8
+F0 "GPIO" 50
+F1 "GPIO.sch" 50
+F2 "ENC1" I R 3500 4450 50
+F3 "ENC2" I R 3500 4550 50
+F4 "ENC_BUTTON" I R 3500 4650 50
+F5 "GPIO_1" I R 3500 4800 50
+F6 "GPIO_2" I R 3500 4900 50
+F7 "GPIO_3" I R 3500 5000 50
+F8 "GPIO_4" I R 3500 5100 50
+F9 "GPIO_5" I R 3500 5200 50
+F10 "GPIO_6" I R 3500 5300 50
+F11 "GPIO_7" I R 3500 5400 50
+F12 "GPIO_8" I R 3500 5500 50
+F13 "GPIO_9" I R 3500 5600 50
+F14 "GPIO_10" I R 3500 5700 50
+F15 "GPIO_11" I R 3500 5800 50
+F16 "GPIO_12" I R 3500 5900 50
+$EndSheet
+Wire Wire Line
+	5000 4450 3500 4450
+Wire Wire Line
+	3500 4550 5000 4550
+Wire Wire Line
+	5000 4650 3500 4650
+Wire Wire Line
+	5000 4800 3500 4800
+Wire Wire Line
+	3500 4900 5000 4900
+Wire Wire Line
+	5000 5000 3500 5000
+Wire Wire Line
+	3500 5100 5000 5100
+Wire Wire Line
+	5000 5200 3500 5200
+Wire Wire Line
+	3500 5300 5000 5300
+Wire Wire Line
+	5000 5400 3500 5400
+Wire Wire Line
+	3500 5500 5000 5500
+Wire Wire Line
+	5000 5600 3500 5600
+Wire Wire Line
+	3500 5700 5000 5700
+Wire Wire Line
+	5000 5800 3500 5800
+Wire Wire Line
+	3500 5900 5000 5900
+Wire Wire Line
+	3500 3150 5000 3150
+Wire Wire Line
+	5000 3250 3500 3250
+Wire Wire Line
+	8500 5200 7500 5200
+Wire Wire Line
+	8500 1450 7500 1450
+Wire Wire Line
+	7500 3100 8500 3100
 $Sheet
 S 5000 1000 2500 5000
@@
 F72 "Diag_LED_1" I R 7500 5200 50
 F73 "BUZZER_ON" I R 7500 1450 50
-$EndSheet
-Wire Wire Line
-	8500 1600 7500 1600
-Wire Wire Line
-	7500 1700 8500 1700
-Wire Wire Line
-	8500 1850 7500 1850
-Wire Wire Line
-	7500 1950 8500 1950
-Wire Wire Line
-	8500 2100 7500 2100
-Wire Wire Line
-	7500 2200 8500 2200
-Wire Wire Line
-	8500 2300 7500 2300
-Wire Wire Line
-	7500 2450 8500 2450
-Wire Wire Line
-	8500 2550 7500 2550
-Wire Wire Line
-	8500 3600 7500 3600
-Wire Wire Line
-	7500 3700 8500 3700
-Wire Wire Line
-	8500 2700 7500 2700
-Wire Wire Line
-	7500 2800 8500 2800
-Wire Wire Line
-	8500 1100 7500 1100
-Wire Wire Line
-	5000 2750 3500 2750
-Wire Wire Line
-	5000 2850 3500 2850
-Wire Wire Line
-	8500 5650 7500 5650
-Wire Wire Line
-	7500 5550 8500 5550
-Wire Wire Line
-	8500 5450 7500 5450
-Wire Wire Line
-	7500 5350 8500 5350
-Wire Wire Line
-	8500 5100 7500 5100
-Wire Wire Line
-	7500 5000 8500 5000
-Wire Wire Line
-	8500 4900 7500 4900
-Wire Wire Line
-	7500 4800 8500 4800
-Wire Wire Line
-	8500 4700 7500 4700
-Wire Wire Line
-	7500 4600 8500 4600
-Wire Wire Line
-	8500 3950 7500 3950
-Wire Wire Line
-	7500 3850 8500 3850
-Wire Wire Line
-	5000 3350 3500 3350
-Wire Wire Line
-	3500 3450 5000 3450
-Wire Wire Line
-	5000 3550 3500 3550
-Wire Wire Line
-	3500 3650 5000 3650
-Wire Wire Line
-	5000 3750 3500 3750
-Wire Wire Line
-	3500 3850 5000 3850
-Wire Wire Line
-	8500 2950 7500 2950
-$Sheet
-S 2500 4350 1000 1650
-U 5F25F1A8
-F0 "GPIO" 50
-F1 "GPIO.sch" 50
-F2 "ENC1" I R 3500 4450 50
-F3 "ENC2" I R 3500 4550 50
-F4 "ENC_BUTTON" I R 3500 4650 50
-F5 "GPIO_1" I R 3500 4800 50
-F6 "GPIO_2" I R 3500 4900 50
-F7 "GPIO_3" I R 3500 5000 50
-F8 "GPIO_4" I R 3500 5100 50
-F9 "GPIO_5" I R 3500 5200 50
-F10 "GPIO_6" I R 3500 5300 50
-F11 "GPIO_7" I R 3500 5400 50
-F12 "GPIO_8" I R 3500 5500 50
-F13 "GPIO_9" I R 3500 5600 50
-F14 "GPIO_10" I R 3500 5700 50
-F15 "GPIO_11" I R 3500 5800 50
-F16 "GPIO_12" I R 3500 5900 50
-$EndSheet
-Wire Wire Line
-	5000 4450 3500 4450
-Wire Wire Line
-	3500 4550 5000 4550
-Wire Wire Line
-	5000 4650 3500 4650
-Wire Wire Line
-	5000 4800 3500 4800
-Wire Wire Line
-	3500 4900 5000 4900
-Wire Wire Line
-	5000 5000 3500 5000
-Wire Wire Line
-	3500 5100 5000 5100
-Wire Wire Line
-	5000 5200 3500 5200
-Wire Wire Line
-	3500 5300 5000 5300
-Wire Wire Line
-	5000 5400 3500 5400
-Wire Wire Line
-	3500 5500 5000 5500
-Wire Wire Line
-	5000 5600 3500 5600
-Wire Wire Line
-	3500 5700 5000 5700
-Wire Wire Line
-	5000 5800 3500 5800
-Wire Wire Line
-	3500 5900 5000 5900
-Wire Wire Line
-	3500 3150 5000 3150
-Wire Wire Line
-	5000 3250 3500 3250
-Wire Wire Line
-	8500 5200 7500 5200
-Wire Wire Line
-	8500 1450 7500 1450
+F74 "Diag_LED_8" I R 7500 3100 50
+$EndSheet
 $EndSCHEMATC
