File: BodyComputer/BodyComputer/GPIO.sch (KiCad schematic (older format))
At the start: 77 parts

Commit message: Update due to moving to another computer. Updated Schematic, Print-outs, PCB in development
Parts:
- D44, D45, D46, D47, D48, D49, D50, D51, D52, D53, D54, D55: renamed from D?; footprint (none) -> Diode_SMD:D_SOD-323_HandSoldering
- J32: renamed from J?; footprint (none) -> SamacSys_Parts:SHDR3W95P0X500_1X3_1620X900X1280P
- gave numbers to parts that had none: 64
Other:
- note removed: "cos"
