File: DRL_Driver/DRL_Driver/DRL_Driver.sch (KiCad schematic (older format))
At the start: 32 parts, among them K1 LEG1A-12, Q1 BC817, Q2 BC817, Q3 IRF5305PBF, U1 4966, U2 4966, U3 4966, U4 4966, U5 4966, U6 4966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

Commit message: Printouts update - small changes in resistors values
Parts:
- R3: value 10k -> 100k
- R7: value 100 -> NULL
Changed lines of the file:
@@
 P 7400 3750
 F 0 "R7" V 7193 3750 50  0000 C CNN
-F 1 "100" V 7284 3750 50  0000 C CNN
+F 1 "NULL" V 7284 3750 50  0000 C CNN
 F 2 "Resistor_SMD:R_0805_2012Metric" V 7330 3750 50  0001 C CNN
 F 3 "~" H 7400 3750 50  0001 C CNN
@@
 P 6500 4250
 F 0 "R3" V 6293 4250 50  0000 C CNN
-F 1 "10k" V 6384 4250 50  0000 C CNN
+F 1 "100k" V 6384 4250 50  0000 C CNN
 F 2 "Resistor_SMD:R_0805_2012Metric" V 6430 4250 50  0001 C CNN
 F 3 "~" H 6500 4250 50  0001 C CNN
