File: MOSFET_Rail/MOSFET_Rail/MOSFET_Rail.sch (KiCad schematic (older format))
At the start: 31 parts, among them J1 Screw_Terminal_01x02, J2 Screw_Terminal_01x02, J3 Screw_Terminal_01x02, Q1 BC817, Q11 IRF5305PBF, Q13 BC817, Q15 IRF5305PBF, Q3 IRF5305PBF, Q5 BC817, Q7 IRF5305PBF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

Commit message: Printouts update - small changes in resistors values
Parts:
- R1, R13, R19, R7: value 4,7k -> 100k
- R11, R17, R23, R5: value 100 -> 0
Changed lines of the file:
@@
 P 1800 1450
 F 0 "R5" V 2000 1400 50  0000 L CNN
-F 1 "100" V 1900 1400 50  0000 L CNN
+F 1 "0" V 1900 1400 50  0000 L CNN
 F 2 "Resistor_SMD:R_0805_2012Metric" V 1730 1450 50  0001 C CNN
 F 3 "~" H 1800 1450 50  0001 C CNN
@@
 P 1050 1450
 F 0 "R1" H 900 1400 50  0000 C CNN
-F 1 "4,7k" H 900 1500 50  0000 C CNN
+F 1 "100k" H 900 1500 50  0000 C CNN
 F 2 "Resistor_SMD:R_0805_2012Metric" V 980 1450 50  0001 C CNN
 F 3 "~" H 1050 1450 50  0001 C CNN
@@
 P 4300 1450
 F 0 "R11" V 4500 1400 50  0000 L CNN
-F 1 "100" V 4400 1400 50  0000 L CNN
+F 1 "0" V 4400 1400 50  0000 L CNN
 F 2 "Resistor_SMD:R_0805_2012Metric" V 4230 1450 50  0001 C CNN
 F 3 "~" H 4300 1450 50  0001 C CNN
@@
 P 3550 1450
 F 0 "R7" H 3400 1400 50  0000 C CNN
-F 1 "4,7k" H 3400 1500 50  0000 C CNN
+F 1 "100k" H 3400 1500 50  0000 C CNN
 F 2 "Resistor_SMD:R_0805_2012Metric" V 3480 1450 50  0001 C CNN
 F 3 "~" H 3550 1450 50  0001 C CNN
@@
 P 6800 1450
 F 0 "R17" V 7000 1400 50  0000 L CNN
-F 1 "100" V 6900 1400 50  0000 L CNN
+F 1 "0" V 6900 1400 50  0000 L CNN
 F 2 "Resistor_SMD:R_0805_2012Metric" V 6730 1450 50  0001 C CNN
 F 3 "~" H 6800 1450 50  0001 C CNN
@@
 P 6050 1450
 F 0 "R13" H 5900 1400 50  0000 C CNN
-F 1 "4,7k" H 5900 1500 50  0000 C CNN
+F 1 "100k" H 5900 1500 50  0000 C CNN
 F 2 "Resistor_SMD:R_0805_2012Metric" V 5980 1450 50  0001 C CNN
 F 3 "~" H 6050 1450 50  0001 C CNN
@@
 P 9300 1450
 F 0 "R23" V 9500 1400 50  0000 L CNN
-F 1 "100" V 9400 1400 50  0000 L CNN
+F 1 "0" V 9400 1400 50  0000 L CNN
 F 2 "Resistor_SMD:R_0805_2012Metric" V 9230 1450 50  0001 C CNN
 F 3 "~" H 9300 1450 50  0001 C CNN
@@
 P 8550 1450
 F 0 "R19" H 8400 1400 50  0000 C CNN
-F 1 "4,7k" H 8400 1500 50  0000 C CNN
+F 1 "100k" H 8400 1500 50  0000 C CNN
 F 2 "Resistor_SMD:R_0805_2012Metric" V 8480 1450 50  0001 C CNN
 F 3 "~" H 8550 1450 50  0001 C CNN
