File: BodyComputer/BodyComputer_v2/BodyComputer_v2/Memory.sch (KiCad schematic (older format))
At the start: 15 parts

Commit message: Finished board design. Schematic names improvements needed.
Parts:
- added C306: 100n, Capacitor_SMD:C_0402_1005Metric, symbol Device:C_Small
- added U303: FRAM_MB85RC16, Package_SO:SOP-8_3.9x4.9mm_P1.27mm, symbol 00_MY_ELEMENTS:FRAM_MB85RC16
- C301, C302, C303, C304, C305: renamed from C?; footprint Capacitor_SMD:C_0603_1608Metric -> Capacitor_SMD:C_0402_1005Metric
- D301: renamed from D?; value LED -> LED_RED
- gave numbers to parts that had none: 9
Connections:
- net +3V3: now also C306.1, U303.8 (VDD)
- net GND: now also C306.2, U303.4 (GND)
- new net FRAM_SCL: U303.6 (SCL)
- new net FRAM_SDA: U303.5 (SDA)
- new net FRAM_WP: U303.7 (WP)
Other:
- note added: "FRAM memory"
