File: BodyComputer/BodyComputer_v2/BodyComputer_v2/Peripherals.sch (KiCad schematic (older format))
At the start: 53 parts

Commit message: Finished board design. Schematic names improvements needed.
Parts:
- removed C? (x2): 100n, Capacitor_SMD:C_0603_1608Metric, symbol Device:C_Small
- added D405: LED_YELLOW, LED_SMD:LED_0603_1608Metric, symbol Device:LED
- added J404: USB_B_Mini, Connector_USB:USB_Mini-B_Lumberg_2486_01_Horizontal, symbol Connector:USB_B_Mini
- added J405: PinHeader, Connector_PinHeader_2.54mm:PinHeader_1x01_P2.54mm_Vertical, symbol Connector_Generic:Conn_01x01
- added R412: 1k, Resistor_SMD:R_0402_1005Metric, symbol Device:R_Small
- C401, C404, C405, C406, C407, C408, C409, C410, C411, C412: renamed from C?; footprint Capacitor_SMD:C_0603_1608Metric -> Capacitor_SMD:C_0402_1005Metric
- D401, D402, D403, D406: renamed from D?; value LED -> LED_RED
- D404, D407: renamed from D?; value LED -> LED_YELLOW
- R413: renamed from R?; value 10k -> 4k7
- gave numbers to parts that had none: 34
Connections:
- net +3V3: now also J402.3 (Pin_3), J402.5 (Pin_5), J402.7 (Pin_7)
- net A0_NODE: now also J407.2 (Pin_2); no longer J407.7 (Pin_7)
- net CLK_NODE: now also J407.7 (Pin_7); no longer J407.9 (Pin_9)
- net CMD_NODE: now also J407.10 (Pin_10); no longer J407.8 (Pin_8)
- net D1_NODE: now also J406.1 (Pin_1); no longer J406.2 (Pin_2)
- net D2_NODE: now also J406.3 (Pin_3); no longer J406.4 (Pin_4)
- net D3_NODE: now also J406.5 (Pin_5); no longer J406.6 (Pin_6)
- net D4_NODE: now also J406.7 (Pin_7); no longer J406.8 (Pin_8)
- net D5_NODE: now also J406.9 (Pin_9); no longer J406.10 (Pin_10)
- net D6_NODE: now also J406.10 (Pin_10); no longer J406.9 (Pin_9)
- net GND: now also J406.4 (Pin_4), D405.1 (K), J404.4 (ID), J404.5 (GND), J404.6 (Shield); no longer J406.3 (Pin_3)
- net NODEMCU_Power: now also J406.2 (Pin_2); no longer J406.1 (Pin_1)
- net RX_NODE: now also J406.8 (Pin_8); no longer J406.7 (Pin_7)
- net SD0_NODE: now also J407.9 (Pin_9); no longer J407.10 (Pin_10)
- net SD1_NODE: now also J407.8 (Pin_8); no longer J407.6 (Pin_6)
- net SD2_NODE: now also J407.6 (Pin_6); no longer J407.4 (Pin_4)
- net SD3_NODE: now also J407.4 (Pin_4); no longer J407.2 (Pin_2)
- net TX_NODE: now also J406.6 (Pin_6); no longer J406.5 (Pin_5)
- net USB_DN: now also J404.2 (D-); no longer J403.2 (D-)
- net USB_DP: now also J404.3 (D+); no longer J403.3 (D+)
- net at J403.1 (VBUS): now also R412.1; no longer R411.1
- net EXTERNAL_RESET: no longer names the net of R413.2, R414.1, SW401.2
- net EXTERNAL_RESET: now also J405.1 (Pin_1)
- net USB_ID renamed USB_BTLD_ID
- new net: J404.1 (VBUS), R411.1
- new net: D405.2 (A), R412.2
- new net USB_BTLD_DN: J403.2 (D-)
- new net USB_BTLD_DP: J403.3 (D+)
Other:
- note added: "USB for BTLD"
- moved on the sheet: BZ401, J402, J403, Q407, R410
