File: BodyComputer/BodyComputer_v2/BodyComputer_v2/PowerSupply.sch (KiCad schematic (older format))
At the start: 47 parts

Commit message: Second version of the body computer - WIP
Parts:
- removed L? (x2): SRN6045TA-6R8M, SRN6045TA-6R8M, symbol SamacSys_Parts:SRN6045TA-6R8M
- added C? (x8): 100n, Capacitor_SMD:C_0603_1608Metric, symbol Device:C_Small
- added C? (x2): 10u, Capacitor_SMD:C_0805_2012Metric, symbol Device:C_Small
- added C? (x2): 1u, Capacitor_SMD:C_0402_1005Metric, symbol Device:C_Small
- added D? (x4): LED, LED_SMD:LED_0603_1608Metric, symbol Device:LED
- added D? (x2): D_Zener, Diode_SMD:D_MiniMELF, symbol Device:D_Zener
- added D? (x2): D, Diode_SMD:D_SMA, symbol Device:D
- added F?: Fuse, SamacSys_Parts:FuseHolder22mm, symbol Device:Fuse
- added L? (x10): L, Inductor_SMD:L_0603_1608Metric, symbol Device:L
- added L? (x2): L, 00_MY_ELEMENTS:COIL_WPN4020H2R2MT, symbol Device:L
- added R?: 470, Resistor_SMD:R_0402_1005Metric, symbol Device:R_Small
- added R? (x8): 1k, Resistor_SMD:R_0402_1005Metric, symbol Device:R_Small
- added R? (x2): 3k6, Resistor_SMD:R_0402_1005Metric, symbol Device:R_Small
- added R? (x3): 10k, Resistor_SMD:R_0402_1005Metric, symbol Device:R_Small
- added R? (x5): 4k7, Resistor_SMD:R_0402_1005Metric, symbol Device:R_Small
- added TH? (x3): NTC, Resistor_SMD:R_0402_1005Metric, symbol Device:Thermistor_NTC
- C? (x9): LCSC (none) -> C15850
- D?: footprint (none) -> Diode_SMD:D_SMA; LCSC (none) -> C22452
- D?: footprint (none) -> Diode_SMD:D_SMB
- U?: LCSC (none) -> C43590
Connections:
- net +12V: now also R?.1, R?.1
- net +3V3: now also C?.1, C?.1, C?.1, C?.2, C?.2, C?.2, L?.2, L?.2, L?.2, L?.2, L?.2, R?.1, R?.1, TH?.1, TH?.1, TH?.1; no longer C?.1, C?.1, C?.1, C?.1, C?.1, C?.1, C?.1, C?.1, C?.1, R?.2, R?.2, R?.2, U?.14 (VOS)
- net +5V: now also C?.1, C?.1, C?.1, C?.2, C?.2, C?.2, L?.2, L?.2, L?.2, L?.2, L?.2, R?.1, R?.1; no longer C?.1, C?.1, C?.1, C?.1, C?.1, C?.1, C?.1, C?.1, C?.1, R?.2, R?.2, R?.2, U?.14 (VOS)
- net +VDC: no longer J?.2 (Pin_2)
- net GND: now also C?.2, C?.2, C?.2, C?.2, C?.2, C?.2, D?.1 (K), D?.1 (K), D?.1 (K), D?.1 (K), D?.2 (A), D?.2 (A), R?.2, R?.2, R?.2, R?.2, R?.2, R?.2
- net at U?.1 (SW), U?.2 (SW), U?.3 (SW): now also L?.1 (x2)
- new net: D?.2 (A), R?.2 (x4)
- new net: C?.1, R?.1, R?.2, TH?.2 (x3)
- new net: C?.1, R?.1, R?.2, R?.2
- new net: C?.1, D?.1 (K), R?.1, R?.2, R?.2 (x2)
- new net: C?.1, C?.1, C?.1, C?.1, C?.1, C?.1, C?.1, C?.1, C?.1, L?.1, L?.1, L?.1, L?.1, L?.1, L?.2, R?.2, R?.2, R?.2, U?.14 (VOS) (x2)
- new net: D?.2 (A), D?.2 (A), F?.1
- new net ADC_3V3: R?.1
- new net ADC_5V: R?.1
- new net ADC_BOARD_TEMP_1: R?.1
- new net ADC_BOARD_TEMP_2: R?.1
- new net ADC_BOARD_TEMP_3: R?.1
- new net ADC_VIN: R?.1
- new net V_CRUISE_CONTROL: R?.1
- new net V_POWER: D?.1 (K), D?.1 (K)
- new net Vdrive: F?.2, J?.2 (Pin_2)
Other:
- note added: "Input Voltage"
- note added: "Temperature\nMonitoring"
- note added: "Voltage Indication"
- note added: "Voltage\nMonitoring"
- moved on the sheet: C?, D?, F?, J?, R?, U?

Commit message: Finished board design. Schematic names improvements needed.
Parts:
- removed D? (x2): D_Zener, Diode_SMD:D_MiniMELF, symbol Device:D_Zener
- removed L? (x2): L, Inductor_SMD:L_0603_1608Metric, symbol Device:L
- added TP201, TP202, TP204: TestPoint, Connector_PinHeader_2.54mm:PinHeader_1x01_P2.54mm_Vertical, symbol Connector:TestPoint_Flag
- C203, C204, C205, C208, C229, C232, C233, C234, C235, C236, C237, C238: renamed from C?; footprint Capacitor_SMD:C_0603_1608Metric -> Capacitor_SMD:C_0402_1005Metric
- D201, D202, D203, D204: renamed from D?; value LED -> LED_YELLOW
- gave numbers to parts that had none: 80
Connections:
- net V_CRUISE_CONTROL is gone; now on net V_POWER: R205.1
- net +3V3: now also TP201.1; no longer C227.2, C228.2, C229.2
- net +5V: now also TP202.1; no longer C230.2, C231.2, C232.2
- net ADC_3V3: now also C233.1
- net ADC_5V: now also C234.1
- net ADC_BOARD_TEMP_1: now also C236.1
- net ADC_BOARD_TEMP_2: now also C237.1
- net ADC_BOARD_TEMP_3: now also C238.1
- net ADC_VIN: now also C235.1
- net GND: now also C227.2, C228.2, C229.2, C230.2, C231.2, C232.2, TP204.1
- net at R226.2, R229.1, TH201.2: no longer C236.1
- net at R227.2, R230.1, TH202.2: no longer C237.1
- net at R228.2, R231.1, TH203.2: no longer C238.1
- net at R217.2, R220.2, R221.1: no longer C233.1
- net at R218.2, R222.2, R223.1: no longer C234.1
- net at R219.2, R224.2, R225.1: no longer C235.1
Other:
- note added: "Near 3V3 DC/DC"
- note added: "Near 5V DC/DC"
- note added: "Near Cruise Control\nDriver"
- note added: "Place NTCs close to:\n3V3 DC/DC\n5V DC/DC\nCruise Control driver"
- moved on the sheet: C233, C234, C235, C236, C237, C238, R226, R227, R228, R229, R230, R231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
