File: BodyComputer/BodyComputer_v2/BodyComputer_v2/Controls.sch (KiCad schematic (older format))
At the start: 40 parts

Commit message: Finished board design. Schematic names improvements needed.
Parts:
- removed C? (x2): 100n, Capacitor_SMD:C_0603_1608Metric, symbol Device:C_Small
- removed C? (x2): 10u, Capacitor_SMD:C_0805_2012Metric, symbol Device:C_Small
- removed D? (x4): LED, LED_SMD:LED_0603_1608Metric, symbol Device:LED
- removed R? (x4): 3k6, Resistor_SMD:R_0402_1005Metric, symbol Device:R_Small
- added C705, C708, C709: 100n, Capacitor_SMD:C_0402_1005Metric, symbol Device:C_Small
- added C712, C715: 10u, Capacitor_SMD:C_0805_2012Metric, symbol Device:C_Small
- added D701, D704, D705: 3V3, Diode_SMD:D_MiniMELF, symbol Device:D_Zener
- added D702, D703, D706, D713, D714, D715, D716: D, Diode_SMD:D_SOD-123, symbol Device:D
- added J701, J702, J703, J704: DB9_Female_MountingHoles, Connector_Dsub:DSUB-9_Female_Horizontal_P2.77x2.84mm_EdgePinOffset7.70mm_Housed_MountingHolesOffset9.12mm, symbol Connector:DB9_Female_MountingHoles
- added K701, K702, K703, K704, K705, K706, K707: RELAY_G5NB-1A-E-DC5V, 00_MY_ELEMENTS:G5NB1A4DC5, symbol 00_MY_ELEMENTS:RELAY_G5NB-1A-E-DC5V
- added Q705, Q706, Q709, Q714, Q715, Q722, Q723, Q724, Q725, Q727, Q728: NPN, Package_TO_SOT_SMD:SOT-23, symbol Device:Q_NPN_BEC
- added Q712, Q713, Q719, Q720, Q721: Q_NMOS_GSD, Package_TO_SOT_SMD:SOT-23, symbol Device:Q_NMOS_GSD
- added Q716, Q726: APM4953, Package_SO:SOP-8_3.76x4.96mm_P1.27mm, symbol 00_MY_ELEMENTS:APM4953
- added R703, R713, R714: 10k, Resistor_SMD:R_0402_1005Metric, symbol Device:R_Small
- added R704, R707, R708, R719, R720, R721, R728, R729, R730, R731, R732, R733, R741, R742, R743, R746, R747, R748, R749, R750, R751, R754, R755: 1k, Resistor_SMD:R_0402_1005Metric, symbol Device:R_Small
- added R724, R725, R736, R737, R738: 22, Resistor_SMD:R_0402_1005Metric, symbol Device:R_Small
- Q710, Q711, Q717, Q718: renamed from Q?; footprint (none) -> Package_TO_SOT_SMD:SOT-23
- gave numbers to parts that had none: 24
Connections:
- net GND: now also C705.2, C708.2, C709.2, C712.2, C715.2, D701.2 (A), D704.2 (A), D705.2 (A), J701.0 (PAD), J702.0 (PAD), J703.0 (PAD), J704.0 (PAD), J704.3, Q705.2 (E), Q706.2 (E), Q709.2 (E), Q712.2 (S), Q713.2 (S), Q714.2 (E), Q715.2 (E), Q719.2 (S), Q720.2 (S), Q721.2 (S), Q722.2 (E), Q723.2 (E), Q724.2 (E), Q725.2 (E), Q727.2 (E), Q728.2 (E), R703.2, R728.2, R729.2, R741.2, R742.2, R743.2
- net PWM_MOS_N_IN_1: now also J703.1
- net PWM_MOS_N_IN_2: now also J703.6
- net PWM_MOS_N_IN_3: now also J703.2
- net PWM_MOS_N_IN_4: now also J703.7
- net PWM_MOS_P_OUT_1: now also J702.6
- net PWM_MOS_P_OUT_2: now also J702.1
- net PWM_MOS_P_OUT_3: now also J702.2
- net PWM_MOS_P_OUT_4: now also J702.7
- net V_POWER: now also C712.1, C715.1, K701.2 (COM), K702.2 (COM), K703.2 (COM), Q716.1 (S1), Q716.3 (S2), Q726.1 (S1), Q726.3 (S2), R732.1, R733.1, R750.1, R751.1
- new net: Q712.1 (G), R724.2, R728.1
- new net: Q719.1 (G), R736.2, R741.1
- new net: Q713.1 (G), R725.2, R729.1
- new net: Q720.1 (G), R737.2, R742.1
- new net: Q721.1 (G), R738.2, R743.1
- new net: D713.2 (A), K704.4 (COIL_2), Q724.3 (C)
- new net: Q724.1 (B), R748.2
- new net: D715.2 (A), K706.4 (COIL_2), Q727.3 (C)
- new net: Q727.1 (B), R754.2
- new net: D714.2 (A), K705.4 (COIL_2), Q725.3 (C)
- new net: Q725.1 (B), R749.2
- new net: D716.2 (A), K707.4 (COIL_2), Q728.3 (C)
- new net: Q728.1 (B), R755.2
- new net: D702.2 (A), K701.4 (COIL_2), Q705.3 (C)
- new net: Q705.1 (B), R707.2
- new net: D706.2 (A), K703.4 (COIL_2), Q709.3 (C)
- new net: Q709.1 (B), R721.2
- new net: D703.2 (A), K702.4 (COIL_2), Q706.3 (C)
- new net: Q706.1 (B), R708.2
- new net: Q714.1 (B), R730.2
- new net: Q714.3 (C), Q716.2 (G1), R732.2
- new net: Q715.3 (C), Q716.4 (G2), R733.2
- new net: Q715.1 (B), R731.2
- new net: Q722.1 (B), R746.2
- new net: Q722.3 (C), Q726.2 (G1), R750.2
- new net: Q723.3 (C), Q726.4 (G2), R751.2
- new net: Q723.1 (B), R747.2
- new net +3V3: R713.2, R714.2
- new net +5V: D702.1 (K), D703.1 (K), D706.1 (K), D713.1 (K), D714.1 (K), D715.1 (K), D716.1 (K), K701.1 (COIL_1), K702.1 (COIL_1), K703.1 (COIL_1), K704.1 (COIL_1), K705.1 (COIL_1), K706.1 (COIL_1), K707.1 (COIL_1)
- new net IN_WIPERS_FAST: C709.1, D705.1 (K), R714.1, R720.1
- new net IN_WIPERS_FAST_SIG: J701.6, R720.2
- new net IN_WIPERS_ON: C705.1, D701.1 (K), R703.1, R704.1
- new net IN_WIPERS_ON_SIG: J701.1, R704.2
- new net IN_WIPERS_SLOW: C708.1, D704.1 (K), R713.1, R719.1
- new net IN_WIPERS_SLOW_SIG: J701.2, R719.2
- new net MOS_P_ON_5: R730.1
- new net MOS_P_ON_6: R731.1
- new net MOS_P_ON_7: R746.1
- new net MOS_P_ON_8: R747.1
- new net MOS_P_OUT_5: J702.8, Q716.7 (D1_1), Q716.8 (D1_2)
- new net MOS_P_OUT_6: J702.4, Q716.5 (D2_1), Q716.6 (D2_2)
- new net MOS_P_OUT_7: J702.5, Q726.7 (D1_1), Q726.8 (D1_2)
- new net MOS_P_OUT_8: J702.9, Q726.5 (D2_1), Q726.6 (D2_2)
- new net PWM_MOS_N_IN_5: J703.3, Q712.3 (D)
- new net PWM_MOS_N_IN_6: J703.8, Q719.3 (D)
- new net PWM_MOS_N_IN_7: J703.4, Q713.3 (D)
- new net PWM_MOS_N_IN_8: J703.9, Q720.3 (D)
- new net PWM_MOS_N_IN_9: J703.5, Q721.3 (D)
- new net PWM_MOS_N_ON_5: R724.1
- new net PWM_MOS_N_ON_6: R736.1
- new net PWM_MOS_N_ON_7: R725.1
- new net PWM_MOS_N_ON_8: R737.1
- new net PWM_MOS_N_ON_9: R738.1
- new net RELAY_IN_1: J704.1, K704.2 (COM)
- new net RELAY_IN_2: J704.2, K706.2 (COM)
- new net RELAY_IN_3: J704.4, K705.2 (COM)
- new net RELAY_IN_4: J704.5, K707.2 (COM)
- new net RELAY_ON_1: R748.1
- new net RELAY_ON_2: R754.1
- new net RELAY_ON_3: R749.1
- new net RELAY_ON_4: R755.1
- new net RELAY_OUT_1: J704.6, K704.3 (NO)
- new net RELAY_OUT_2: J704.7, K706.3 (NO)
- new net RELAY_OUT_3: J704.8, K705.3 (NO)
- new net RELAY_OUT_4: J704.9, K707.3 (NO)
- new net WIPERS_SIG2_ON: R707.1
- new net WIPERS_SIG2_ON_SIG: J701.3, K701.3 (NO)
- new net WIPERS_SIG3_ON: R721.1
- new net WIPERS_SIG3_ON_SIG: J701.5, K703.3 (NO)
- new net WIPERS_SIG5_ON: R708.1
- new net WIPERS_SIG5_ON_SIG: J701.4, K702.3 (NO)
- no-connect marks 0 -> 4
Other:
- note added: "MOSFET N, Channels 1-7"
- note added: "MOSFET P, Channel 5 and 6"
- note added: "MOSFET P, Channel 7 and 8"
- moved on the sheet: Q710, Q711, Q717, Q718, R722, R723, R726, R727, R734, R735, R739, R740

Commit message: Signals naming improvements
Connections:
- net MOS_P_ON_5 renamed PWM_MOS_P_ON_5
- net MOS_P_ON_7 renamed PWM_MOS_P_ON_7
- net MOS_P_ON_8 renamed PWM_MOS_P_ON_8
- net MOS_P_OUT_5 renamed PWM_MOS_P_OUT_5
- net MOS_P_OUT_7 renamed PWM_MOS_P_OUT_7
- net MOS_P_OUT_8 renamed PWM_MOS_P_OUT_8
- net PWM_MOS_P_ON_2 renamed MOS_P_ON_2
- net PWM_MOS_P_ON_3 renamed MOS_P_ON_3
- net PWM_MOS_P_ON_4 renamed MOS_P_ON_4
- net PWM_MOS_P_OUT_2 renamed MOS_P_OUT_2
- net PWM_MOS_P_OUT_3 renamed MOS_P_OUT_3
- net PWM_MOS_P_OUT_4 renamed MOS_P_OUT_4
Other:
- moved on the sheet: C706, C707, C712, Q701, Q702, Q703, Q704, Q707, Q708, Q714, Q715, Q716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
