File: BodyComputer/BodyComputer_v2/BodyComputer_v2/BodyComputer_v2.sch (KiCad schematic (older format))
At the start: 0 parts

Commit message: Final naming changes
Changed lines of the file:
@@
 F13 "ADC_LM35_2_N" I R 3500 3400 50
 F14 "ADC_ACC_POSITION" I R 3500 4650 50
-F15 "ADC_FUEL_POSITION" I R 3500 4750 50
-F16 "ADC_LM35_3_P" I R 3500 3500 50
-F17 "ADC_LM35_3_N" I R 3500 3600 50
-F18 "ADC_LM35_4_N" I R 3500 3800 50
-F19 "ADC_LM35_4_P" I R 3500 3700 50
-F20 "ADC_LM35_5_P" I R 3500 3900 50
-F21 "ADC_LM35_5_N" I R 3500 4000 50
-F22 "ADC_POTENTIOMETER_1" I R 3500 4400 50
-F23 "ADC_RESISTANCE_SENS_1" I R 3500 4150 50
-F24 "ADC_RESISTANCE_SENS_2" I R 3500 4250 50
-F25 "ADC_POTENTIOMETER_2" I R 3500 4500 50
-F26 "IN_BIN_1" I R 3500 6150 50
-F27 "IN_BIN_2" I R 3500 6250 50
-F28 "IN_BIN_3" I R 3500 6350 50
-F29 "IN_BIN_4" I R 3500 6450 50
-F30 "IN_BIN_5" I R 3500 6550 50
-F31 "IN_BIN_6" I R 3500 6650 50
-F32 "IN_BIN_7" I R 3500 6750 50
-F33 "IN_BIN_8" I R 3500 6850 50
-F34 "ADC_MAIN_BATTERY" I R 3500 5050 50
-F35 "ADC_AUX_BATTERY" I R 3500 5150 50
+F15 "ADC_LM35_3_P" I R 3500 3500 50
+F16 "ADC_LM35_3_N" I R 3500 3600 50
+F17 "ADC_LM35_4_N" I R 3500 3800 50
+F18 "ADC_LM35_4_P" I R 3500 3700 50
+F19 "ADC_LM35_5_P" I R 3500 3900 50
+F20 "ADC_LM35_5_N" I R 3500 4000 50
+F21 "ADC_POTENTIOMETER_1" I R 3500 4400 50
+F22 "ADC_RESISTANCE_SENS_1" I R 3500 4150 50
+F23 "ADC_RESISTANCE_SENS_2" I R 3500 4250 50
+F24 "ADC_POTENTIOMETER_2" I R 3500 4500 50
+F25 "IN_BIN_1" I R 3500 6150 50
+F26 "IN_BIN_2" I R 3500 6250 50
+F27 "IN_BIN_3" I R 3500 6350 50
+F28 "IN_BIN_4" I R 3500 6450 50
+F29 "IN_BIN_5" I R 3500 6550 50
+F30 "IN_BIN_6" I R 3500 6650 50
+F31 "IN_BIN_7" I R 3500 6750 50
+F32 "IN_BIN_8" I R 3500 6850 50
+F33 "ADC_MAIN_BATTERY" I R 3500 5050 50
+F34 "ADC_AUX_BATTERY" I R 3500 5150 50
+F35 "ADC_FUEL_LEVEL" I R 3500 4750 50
 $EndSheet
 $Sheet
