File: BodyComputer/BodyComputer_v2/BodyComputer_v2/CruiseControl.sch (KiCad schematic (older format))
At the start: 38 parts

Commit message: Finished board design. Schematic names improvements needed.
Parts:
- removed C?: 100n, Capacitor_SMD:C_0603_1608Metric, symbol Device:C_Small
- removed C?: 10u, Capacitor_SMD:C_0805_2012Metric, symbol Device:C_Small
- C504, C505, C506, C507, C508, C509: renamed from C?; footprint Capacitor_SMD:C_0603_1608Metric -> Capacitor_SMD:C_0402_1005Metric
- D501: renamed from D?; value LED -> LED_RED
- gave numbers to parts that had none: 29
Connections:
- net CRUISE_CONTROL_Power: now also Q502.5 (D2_1), Q502.6 (D2_2); no longer Q502.7 (D1_1), Q502.8 (D1_2)
- net ENC1_BUTTON: now also R522.2; no longer R506.2
- net ENC1_CH_B: now also R506.2; no longer R522.2
- net ENC2_BUTTON: now also R523.2; no longer R507.2
- net ENC2_CH_B: now also R507.2; no longer R523.2
- net GND: now also J501.6, J501.7, J501.8, J501.9; no longer J501.2, J501.3, J501.4, J501.5
- net OUT1_ELECTRO_CLUTCH: now also J501.3; no longer J501.6
- net OUT1_ENGINE: now also J501.2; no longer J501.8
- net OUT2_ELECTRO_CLUTCH: now also J501.4; no longer J501.7
- net OUT2_ENGINE: now also J501.5; no longer J501.9
- net V_POWER: now also Q502.3 (S2); no longer Q502.1 (S1)
- net at Q501.3 (C), R508.2: now also Q502.4 (G2); no longer Q502.2 (G1)
Other:
- moved on the sheet: Q502

Commit message: Final naming changes
Connections:
- net ENC1_BUTTON_IN: now also J502.2, R518.1; no longer J502.6, R501.1
- net ENC1_CH_B_IN: now also J502.6, R501.1; no longer J502.2, R518.1
- net ENC2_BUTTON_IN: now also J502.4, R519.1; no longer J502.9, R502.1
- net ENC2_CH_B_IN: now also J502.9, R502.1; no longer J502.4, R519.1
Changed lines of the file:
@@
 Wire Wire Line
 	3100 8200 2900 8200
-Text Label 1750 8200 2    50   ~ 0
+Text Label 6750 8200 2    50   ~ 0
 ENC1_BUTTON_IN
 $Comp
@@
 Wire Wire Line
 	8100 8200 7900 8200
-Text Label 6750 8200 2    50   ~ 0
+Text Label 1750 8200 2    50   ~ 0
 ENC1_CH_B_IN
 $Comp
@@
 Wire Wire Line
 	3100 9700 2900 9700
-Text Label 1750 9700 2    50   ~ 0
+Text Label 6750 9700 2    50   ~ 0
 ENC2_BUTTON_IN
 $Comp
@@
 Wire Wire Line
 	8100 9700 7900 9700
-Text Label 6750 9700 2    50   ~ 0
+Text Label 1750 9700 2    50   ~ 0
 ENC2_CH_B_IN
 $Comp
@@
 Text Label 4250 8200 2    50   ~ 0
 ENC1_CH_A_IN
-Text Label 5300 6250 2    50   ~ 0
+Text Label 5300 6350 2    50   ~ 0
 ENC2_CH_B_IN
 Wire Wire Line
@@
 Text Label 5300 6450 2    50   ~ 0
 ENC2_CH_A_IN
-Text Label 5300 6350 2    50   ~ 0
+Text Label 5300 6250 2    50   ~ 0
 ENC2_BUTTON_IN
+Text Label 5300 5750 2    50   ~ 0
+ENC1_CH_B_IN
 Text Label 5300 5850 2    50   ~ 0
-ENC1_CH_B_IN
-Text Label 5300 5750 2    50   ~ 0
 ENC1_BUTTON_IN
 Wire Wire Line
