File: BodyComputer/BodyComputer_v2/BodyComputer_v2/Measurements.sch (KiCad schematic (older format))
At the start: 140 parts

Commit message: Finished board design. Schematic names improvements needed.
Parts:
- removed C? (x2): 100n, Capacitor_SMD:C_0603_1608Metric, symbol Device:C_Small
- removed R? (x3): 470, Resistor_SMD:R_0402_1005Metric, symbol Device:R_Small
- C611, C612, C620, C621, C622, C623, C624, C625, C626, C627, C628, C629, C630, C631: renamed from C?; footprint Capacitor_SMD:C_0603_1608Metric -> Capacitor_SMD:C_0402_1005Metric
- gave numbers to parts that had none: 121
Connections:
- net OIL_PRESS_ANALOG_IN is gone; now on net GND: J605.5
- net OPTOCOUPLER_VCC is gone; now on net OPTOCOUPLER_GND: R625.2, R626.2
- net IN_BIN_SIG_1: now also J606.6; no longer J606.1
- net IN_BIN_SIG_2: now also J606.1; no longer J606.6
- net IN_BIN_SIG_6: now also J606.4; no longer J606.8
- net IN_BIN_SIG_7: now also J606.8; no longer J606.4
- net LM35_1_SIG_N: now also J602.2; no longer J602.5
- net LM35_3_SIG_N: now also J602.5; no longer J602.2
Other:
- moved on the sheet: R625, R626

Commit message: Final naming changes
Connections:
- net ADC_FUEL_POSITION renamed ADC_FUEL_LEVEL
Changed lines of the file:
@@
 Brake Pedal Press Signal
 Text HLabel 2750 5500 0    50   Input ~ 0
-ADC_FUEL_POSITION
+ADC_FUEL_LEVEL
 $Comp
 L power:GND #PWR?
@@
 	4050 10050 4050 10350
 Wire Notes Line
-	2950 10350 2950 10050
-Wire Notes Line
-	2950 9750 2950 9450
-Wire Notes Line
 	4450 9450 4450 9750
